File: HARDWARE/MAIN/Pi_grammer_MAIN.sch (EAGLE design)
At the start: 60 parts, among them J1 RASPBERRYPI-B+-GPIO, J2 SPI, Q1 220mA/50V/3.5Ω, Q2 220mA/50V/3.5Ω, Q3 220mA/50V/3.5Ω, Q4 220mA/50V/3.5Ω, Q5 220mA/50V/3.5Ω, U1 AT42QT1010 - UDFN, U2 74LVC4066

Commit message: Changed a 3.3V net flag to a proper "VCC" symbol
Note, this flag was for the 3.3V hitting the resistor for the "POWER" LED.
Changed lines of the file:
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@@
 <?xml version="1.0" encoding="utf-8"?>
 <!DOCTYPE eagle SYSTEM "eagle.dtd">
-<eagle version="7.6.0">
+<eagle version="6.5.0">
 <drawing>
 <settings>
@@
 <part name="FD3" library="SparkFun-Aesthetics" deviceset="FIDUCIAL" device="UFIDUCIAL"/>
 <part name="FD4" library="SparkFun-Aesthetics" deviceset="FIDUCIAL" device="UFIDUCIAL"/>
+<part name="SUPPLY3" library="SparkFun-Aesthetics" deviceset="3.3V" device=""/>
 </parts>
 <sheets>
@@
 <instance part="FD3" gate="G$1" x="254" y="208.28"/>
 <instance part="FD4" gate="G$1" x="251.46" y="210.82"/>
+<instance part="SUPPLY3" gate="G$1" x="223.52" y="353.06"/>
 </instances>
 <busses>
@@
 <wire x1="35.56" y1="347.98" x2="22.86" y2="347.98" width="0.1524" layer="91"/>
 <junction x="22.86" y="347.98"/>
-</segment>
-<segment>
-<pinref part="R1" gate="G$1" pin="2"/>
-<wire x1="226.06" y1="350.52" x2="223.52" y2="350.52" width="0.1524" layer="91"/>
-<label x="223.52" y="350.52" size="1.27" layer="95" rot="R180" xref="yes"/>
 </segment>
 <segment>
@@
 <pinref part="C3" gate="G$1" pin="1"/>
 </segment>
+<segment>
+<pinref part="SUPPLY3" gate="G$1" pin="3.3V"/>
+<pinref part="R1" gate="G$1" pin="2"/>
+<wire x1="226.06" y1="350.52" x2="223.52" y2="350.52" width="0.1524" layer="91"/>
+<wire x1="223.52" y1="350.52" x2="223.52" y2="353.06" width="0.1524" layer="91"/>
+</segment>
 </net>
