File: HARDWARE/HAT/SparkFun_Pi_AVR_Programmer_HAT.brd (EAGLE design)
At the start: 73.7 x 78.7 mm, 60 parts, among them J1 RASPBERRYPI-B+-GPIO, J2 SPI, Q1 220mA/50V/3.5Ω, Q2 220mA/50V/3.5Ω, Q3 220mA/50V/3.5Ω, Q4 220mA/50V/3.5Ω, Q5 220mA/50V/3.5Ω, U1 AT42QT1010 - UDFN, U2 74LVC4066

Commit message: Adjusted silk for new product name
Also updated all silk to sweet buzzard style labels
Parts:
- added U$1: (no value), buzzard_labels:SPARKFUN_PI_AVR_PROGRAMMER_HAT0
- added U$10: (no value), buzzard_labels (5):5V_#PI#8
- added U$11: (no value), buzzard_labels (6):TARGET0
- added U$12: (no value), buzzard_labels (5):MISO1
- added U$13: (no value), buzzard_labels (5):MOSI0
- added U$14: (no value), buzzard_labels (5):SCK2
- added U$15: (no value), buzzard_labels (5):RST3
- added U$16: (no value), buzzard_labels (5):GND4
- added U$18: (no value), buzzard_labels (7):TAP0
- added U$19: (no value), buzzard_labels (7):TO1
- added U$2: (no value), buzzard_labels (2):PROJECT_NAME0
- added U$20: (no value), buzzard_labels (7):PROGRAM2
- added U$21: (no value), buzzard_labels (9):VCC0
- added U$22: (no value), buzzard_labels (8):SUCCESS0
- added U$23: (no value), buzzard_labels (8):FUSE_BITS2
- added U$24: (no value), buzzard_labels (8):FLASH_HEX3
- added U$25: (no value), buzzard_labels (8):LOCK_BITS4
- added U$26: (no value), buzzard_labels (8):SERIAL_UPLOAD5
- added U$3: (no value), buzzard_labels (3):VERSION_#_DATE_#_ETC#0
- added U$4: (no value), buzzard_labels (4):TARGET_LOGIC_SELECT4
- added U$5: (no value), buzzard_labels (4):POWER0
- added U$6: (no value), buzzard_labels (4):STAT1
- added U$7: (no value), buzzard_labels (4):SHUTDOWN2
- added U$8: (no value), buzzard_labels (4):RASPI3
- added U$9: (no value), buzzard_labels (5):3#3V_#PI#7
- moved LOGO1 6.35 mm to (33.4, 66.9)
Other:
- board text removed: "3.3V (PI)"
- board text removed: "5V (PI)"
- board text removed: "FLASH HEX"
- board text removed: "FUSE BITS"
- board text removed: "GND"
- board text removed: "LOCK BITS"
- board text removed: "MISO"
- board text removed: "MOSI"
- board text removed: "POWER"
- board text removed: "PROGRAM"
- board text removed: "PROJECT NAME"
- board text removed: "Pi_grammer"
- board text removed: "RASPI AVR PROGRAMMER"
- board text removed: "RST"
- board text removed: "SCK"
- board text removed: "SERIAL UPLOAD"
- board text removed: "SHUTDOWN RASPI"
- board text removed: "STAT"
- board text removed: "SUCCESS"
- board text removed: "TAP"
- board text removed: "TARGET LOGIC SELECT"
- board text removed: "TARGET VCC"
- board text removed: "TO"
- board text removed: "VCC_T"
- board text removed: "VERSION, DATE, ETC."

Commit message: fixed hatch ground pour under capsense pad
Due to inverted sPlace (silk), it was hard to see that the hatched GND was actually gone. I must have ripped up a "floating" GND trace that connects the hatched GND polygon to the main GND polygon on the botton copper.
Routing:
- net GND: track 1.31 -> 22.7 mm
- net PAD: vias 1 -> 0
Changed lines of the file:
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@@
 <setting verticaltext="up"/>
 </settings>
-<grid distance="0.05" unitdist="inch" unit="inch" style="lines" multiple="1" display="yes" altdistance="0.001" altunitdist="inch" altunit="inch"/>
+<grid distance="0.05" unitdist="inch" unit="inch" style="lines" multiple="1" display="yes" altdistance="0.005" altunitdist="inch" altunit="inch"/>
 <layers>
 <layer number="1" name="Top" color="4" fill="1" visible="yes" active="yes"/>
@@
 <rectangle x1="16.4084" y1="71.12" x2="25.4" y2="73.1647" layer="21"/>
 <rectangle x1="1.27" y1="44.45" x2="44.45" y2="54.61" layer="21"/>
-<rectangle x1="22.545040625" y1="54.61" x2="44.45" y2="56.36768125" layer="21"/>
+<rectangle x1="22.545040625" y1="54.61" x2="44.449996875" y2="56.36768125" layer="21"/>
 <polygon width="0.254" layer="21">
 <vertex x="10.16" y="15.24"/>
@@
 <vertex x="73.66" y="78.74"/>
 <vertex x="73.66" y="0"/>
-<vertex x="20.32" y="0"/>
-<vertex x="20.32" y="19.05"/>
-<vertex x="0" y="19.05"/>
+<vertex x="21.59" y="0"/>
+<vertex x="21.59" y="20.32"/>
+<vertex x="0" y="20.32"/>
 </polygon>
 <polygon width="0.381" layer="1" isolate="0.381">
@@
 <contactref element="U1" pad="4"/>
 <polygon width="0.3048" layer="16" pour="hatch" isolate="0.3048">
-<vertex x="20.32" y="1.27"/>
-<vertex x="1.27" y="1.27"/>
-<vertex x="1.27" y="19.05"/>
-<vertex x="20.32" y="19.05"/>
+<vertex x="21.59" y="0"/>
+<vertex x="2.54" y="0" curve="-90"/>
+<vertex x="0" y="2.54"/>
+<vertex x="0" y="20.32"/>
+<vertex x="21.59" y="20.32"/>
 </polygon>
 <contactref element="D9" pad="C"/>
@@
 <via x="64.389" y="59.563" extent="1-16" drill="0.508"/>
 <via x="65.532" y="56.896" extent="1-16" drill="0.508"/>
+<wire x1="26.44" y1="22.86" x2="12.7" y2="22.86" width="0.254" layer="1"/>
+<wire x1="7.62" y1="22.86" x2="7.62" y2="15.24" width="0.254" layer="16"/>
 </signal>
 <signal name="5V">
@@
 <contactref element="Q1" pad="2"/>
 <contactref element="R13" pad="2"/>
-<wire x1="48.514" y1="41.91" x2="49.657" y2="40.767" width="0.254" layer="1"/>
+<wire x1="48.514" y1="41.91" x2="49.784" y2="40.64" width="0.254" layer="1"/>
 <wire x1="62.5" y1="46.04" x2="59.79" y2="46.04" width="0.254" layer="1"/>
 <wire x1="59.79" y1="46.04" x2="59.69" y2="46.14" width="0.254" layer="1"/>
@@
 <wire x1="55.88" y1="43.18" x2="53.34" y2="40.64" width="0.254" layer="1"/>
 <wire x1="53.34" y1="40.64" x2="49.784" y2="40.64" width="0.254" layer="1"/>
-<wire x1="49.784" y1="40.64" x2="49.657" y2="40.767" width="0.254" layer="1"/>
 </signal>
 <signal name="MISO">
@@
 <vertex x="20.32" y="3.81"/>
 </polygon>
-<via x="19.05" y="12.7" extent="1-16" drill="0.508"/>
 <wire x1="27.09" y1="11.43" x2="20.32" y2="11.43" width="0.254" layer="1"/>
 <wire x1="20.32" y1="11.43" x2="19.05" y2="12.7" width="0.254" layer="1"/>
@@
 <wire x1="68.58" y1="36.83" x2="63.5" y2="36.83" width="0.254" layer="1"/>
 <wire x1="63.5" y1="36.83" x2="61.595" y2="34.925" width="0.254" layer="1"/>
-<wire x1="61.595" y1="34.925" x2="61.595" y2="34.29" width="0.254" layer="1"/>
 <wire x1="61.595" y1="33.44" x2="61.595" y2="30.74" width="0.254" layer="1"/>
 <wire x1="61.175" y1="33.02" x2="61.595" y2="33.44" width="0.254" layer="1"/>
-<wire x1="61.595" y1="33.44" x2="61.595" y2="34.29" width="0.254" layer="1"/>
+<wire x1="61.595" y1="33.44" x2="61.595" y2="34.925" width="0.254" layer="1"/>
 </signal>
 <signal name="PGM_CTRL_T">
